Commit message: Update test.urdf

File: urdf/test.urdf (robot description, URDF)
Before this commit: robot base_robot, 3 links, 2 joints
Links:
- added link wheel_bl/base_link; visual cylinder length=0.05 radius=0.075
- added link wheel_br/base_link; visual cylinder length=0.05 radius=0.075
- link wheel_fl/base_link: geometry visual cylinder length=0.05 radius=0.075
- link wheel_fr/base_link: geometry visual cylinder length=0.05 radius=0.075
Joints:
- added joint wheel_bl/base_joint: type fixed, parent base_link, child wheel_bl/base_link, origin xyz=-0.3 0.35 0.02 rpy=0 1.5708 1.5708
- added joint wheel_br/base_joint: type fixed, parent base_link, child wheel_br/base_link, origin xyz=-0.3 -0.35 0.02 rpy=0 1.5708 1.5708
- joint wheel_fl/base_joint: origin xyz=0.3 -0.335 0.02 rpy=0 1.5708 1.5708 -> xyz=0.3 0.35 0.02 rpy=0 1.5708 1.5708
- joint wheel_fr/base_joint: origin xyz=0.3 -0.335 0.02 rpy=0 1.5708 1.5708 -> xyz=0.3 -0.35 0.02 rpy=0 1.5708 1.5708
